File: Lycheepark/Lycheepark.kicad_pcb (KiCad board)
At the start: 2 copper layers, 33.5 x 32 mm, 21 parts, among them J1 HOST_PROG, J2 USB_CDC, Q1 S8050, U1 ESP32-S3-WROOM-1, U2 AMS1117-3.3

Commit message: Rev 2: init
Parts:
- added TP1: TestPoint, TestPoint:TestPoint_Pad_1.5x1.5mm, F.Cu at (111.4, 128.1)
- added TP2: TestPoint, TestPoint:TestPoint_Pad_1.5x1.5mm, F.Cu at (114.2, 128.1)
- J2, LCD1: moved to B.Cu
- moved D1 23.9 mm to (129.6, 108.7)
- moved R5 10.0 mm to (131.4, 119.5), turned to 0 degrees
- moved C8 9.84 mm to (118.7, 128.9)
- moved R6 7.76 mm to (131.5, 117.3), turned to 0 degrees
- moved C5 6.88 mm to (131.4, 114.8), turned to 0 degrees
- moved C4 4.59 mm to (101.6, 117.0), turned to 90 degrees
- moved R3 4.01 mm to (103.6, 126.7), turned to 180 degrees
- moved C1 2.30 mm to (108.8, 129.2)
- moved C7 2.17 mm to (123.9, 130.2), turned to 180 degrees
- moved LCD1 2.13 mm to (105.0, 116.2), turned to 0 degrees
- moved R2 1.87 mm to (101.7, 123.8)
- moved R4 1.86 mm to (103.8, 123.8)
- moved C6 1.02 mm to (123.9, 127.9), turned to 180 degrees
- moved R1 0.92 mm to (103.8, 110.7)
- moved U2 0.48 mm to (129.7, 126.8)
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Connections:
- U1 pad 17: unconnected-(U1-Pad17) -> SDA
- U1 pad 18: unconnected-(U1-Pad18) -> SCL
Routing:
- net +3V3: track 94.9 -> 118.0 mm
- net STAT_LED: track 9.26 -> 21.0 mm, vias 2 -> 0
- net Net-(J2-PadA5): track 12.6 -> 4.29 mm, vias 2 -> 1
- net +5V: track 28.8 -> 23.4 mm, vias 0 -> 2
- net Net-(J2-PadB5): track 8.43 -> 3.80 mm, vias 2 -> 1
- net USB_DP: track 30.2 -> 26.8 mm, vias 2 -> 1
- net Net-(Q1-Pad1): track 7.38 -> 4.15 mm
- net SCL: track 0.00 -> 3.21 mm
- net Net-(Q1-Pad3): track 2.59 -> 5.49 mm
- net SDA: track 0.00 -> 2.63 mm
- net LEDK: track 8.03 -> 5.79 mm, vias 0 -> 1
- net GND: track 59.2 -> 61.3 mm, vias 204 -> 222
- net EN: track 25.0 -> 23.0 mm
- net DISP_BL: track 11.9 -> 10.1 mm
- net USB_DM: track 28.3 -> 29.3 mm
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Other:
- board size 33.5 x 32 mm -> 33.5 x 31.5 mm
