File: Lycheepark/Lycheepark.kicad_sch (KiCad schematic)
At the start: 21 parts, among them J1 HOST_PROG, J2 USB_CDC, Q1 S8050, U1 ESP32-S3-WROOM-1, U2 AMS1117-3.3

Commit message: Rev 2: init
Parts:
- added TP_SCL1, TP_SDA1: (no value), symbol Connector:TestPoint
Connections:
- net SDA: now reaches U1.17 (GPIO9/TOUCH9/ADC1_CH8/FSPIHD/SUBSPIHD)
- net SDA: now also TP_SDA1.1
- net SCL: now reaches U1.18 (GPIO10/TOUCH10/ADC1_CH9/FSPICS0/FSPIIO4/SUBSPICS0)
- net SCL: now also TP_SCL1.1
- no-connect marks 24 -> 23
Changed lines of the file:
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@@
   )
   (no_connect (at 27.94 31.75))
-  (no_connect (at 27.94 52.07))
-  (no_connect (at 27.94 54.61))
   (no_connect (at 27.94 57.15))
   (no_connect (at 27.94 59.69))
@@
   (no_connect (at 194.31 69.85))
   (no_connect (at 52.07 147.32))
+  (no_connect (at 27.94 36.83))
   (wire (pts (xy 29.21 160.02) (xy 29.21 163.83))
     (stroke (width 0) (type default) (color 0 0 0 0))
@@
     (stroke (width 0) (type default) (color 0 0 0 0))
   )
+  (wire (pts (xy 25.4 54.61) (xy 27.94 54.61))
+    (stroke (width 0) (type default) (color 0 0 0 0))
+  )
   (wire (pts (xy 177.8 134.62) (xy 180.34 134.62))
     (stroke (width 0) (type default) (color 0 0 0 0))
@@
     (stroke (width 0) (type default) (color 0 0 0 0))
   )
+  (wire (pts (xy 27.94 182.88) (xy 31.75 182.88))
+    (stroke (width 0) (type default) (color 0 0 0 0))
+  )
   (polyline (pts (xy 162.56 12.7) (xy 162.56 107.95))
     (stroke (width 0) (type default) (color 0 0 0 0))
   )
+  (wire (pts (xy 25.4 52.07) (xy 27.94 52.07))
+    (stroke (width 0) (type default) (color 0 0 0 0))
+  )
   (wire (pts (xy 264.16 133.35) (xy 264.16 137.16))
     (stroke (width 0) (type default) (color 0 0 0 0))
@@
   )
   (wire (pts (xy 233.68 148.59) (xy 248.92 148.59))
+    (stroke (width 0) (type default) (color 0 0 0 0))
+  )
+  (wire (pts (xy 27.94 193.04) (xy 31.75 193.04))
     (stroke (width 0) (type default) (color 0 0 0 0))
   )
@@
     )
   )
+  (global_label "SCL" (shape input) (at 31.75 193.04 0) (fields_autoplaced)
+    (effects (font (size 1.27 1.27)) (justify left))
+    (property "Intersheet References" "${INTERSHEET_REFS}" (id 0) (at 37.6707 192.9606 0)
+      (effects (font (size 1.27 1.27)) (justify left) hide)
+    )
+  )
   (global_label "BOOT" (shape input) (at 24.13 25.4 180) (fields_autoplaced)
     (effects (font (size 1.27 1.27)) (justify right))
@@
     (property "Intersheet References" "${INTERSHEET_REFS}" (id 0) (at 218.3606 148.4026 90)
       (effects (font (size 1.27 1.27)) (justify right) hide)
+    )
+  )
+  (global_label "SDA" (shape input) (at 31.75 182.88 0) (fields_autoplaced)
+    (effects (font (size 1.27 1.27)) (justify left))
+    (property "Intersheet References" "${INTERSHEET_REFS}" (id 0) (at 37.7312 182.8006 0)
+      (effects (font (size 1.27 1.27)) (justify left) hide)
     )
   )
@@
     )
   )
+  (global_label "SCL" (shape input) (at 25.4 54.61 180) (fields_autoplaced)
+    (effects (font (size 1.27 1.27)) (justify right))
+    (property "Intersheet References" "${INTERSHEET_REFS}" (id 0) (at 19.4793 54.5306 0)
+      (effects (font (size 1.27 1.27)) (justify right) hide)
+    )
+  )
   (global_label "USB_DP" (shape input) (at 66.04 139.7 0) (fields_autoplaced)
     (effects (font (size 1.27 1.27)) (justify left))
@@
     (effects (font (size 1.27 1.27)) (justify right))
     (property "Intersheet References" "${INTERSHEET_REFS}" (id 0) (at 165.4688 69.7706 0)
+      (effects (font (size 1.27 1.27)) (justify right) hide)
+    )
+  )
+  (global_label "SDA" (shape input) (at 25.4 52.07 180) (fields_autoplaced)
+    (effects (font (size 1.27 1.27)) (justify right))
+    (property "Intersheet References" "${INTERSHEET_REFS}" (id 0) (at 19.4188 51.9906 0)
       (effects (font (size 1.27 1.27)) (justify right) hide)
     )
@@
     (pin "2")
   )
+  (symbol (lib_id "Connector:TestPoint") (at 27.94 193.04 90) (unit 1)
+    (in_bom yes) (on_board yes) (fields_autoplaced)
+    (property "Reference" "TP_SCL1" (id 0) (at 24.638 186.69 90))
+    (property "Value" "" (id 1) (at 24.638 189.23 90))
+    (property "Footprint" "" (id 2) (at 27.94 187.96 0)
+      (effects (font (size 1.27 1.27)) hide)
+    )
+    (property "Datasheet" "~" (id 3) (at 27.94 187.96 0)
+      (effects (font (size 1.27 1.27)) hide)
+    )
+    (pin "1")
+  )
   (symbol (lib_id "Device:C_Small") (at 99.06 144.78 0) (unit 1)
     (in_bom yes) (on_board yes)
@@
     (pin "1")
   )
+  (symbol (lib_id "Connector:TestPoint") (at 27.94 182.88 90) (unit 1)
+    (in_bom yes) (on_board yes) (fields_autoplaced)
+    (property "Reference" "TP_SDA1" (id 0) (at 24.638 176.53 90))
+    (property "Value" "" (id 1) (at 24.638 179.07 90))
+    (property "Footprint" "" (id 2) (at 27.94 177.8 0)
+      (effects (font (size 1.27 1.27)) hide)
+    )
+    (property "Datasheet" "~" (id 3) (at 27.94 177.8 0)
+      (effects (font (size 1.27 1.27)) hide)
+    )
+    (pin "1")
+  )
   (symbol (lib_id "Device:R_Small") (at 240.03 82.55 0) (unit 1)
     (in_bom yes) (on_board yes)
@@
       (reference "R6") (unit 1) (value "5.11k") (footprint "Resistor_SMD:R_0805_2012Metric_Pad1.20x1.40mm_HandSolder")
     )
+    (path "/785ef9f2-83dd-4d0e-926f-6bf23b7dbf36"
+      (reference "TP_SCL1") (unit 1) (value "TestPoint") (footprint "TestPoint:TestPoint_Pad_1.5x1.5mm")
+    )
+    (path "/e96f05bb-d53b-45c6-ac4c-12cf857233a5"
+      (reference "TP_SDA1") (unit 1) (value "TestPoint") (footprint "TestPoint:TestPoint_Pad_1.5x1.5mm")
+    )
     (path "/1a76a9f3-b790-4d69-9562-cddac9112333"
